Commit message: Add planner node. App is working

File: workcell_scene_description/urdf/red_ball.urdf (robot description, URDF)
Before this commit: robot red_ball, 1 links, 0 joints
Links:
- link red_ball: geometry collision sphere radius=0.075; visual sphere radius=0.075

Commit message: Update documentation

File: workcell_scene_description/urdf/red_ball.urdf (robot description, URDF)
Before this commit: robot red_ball, 1 links, 0 joints
Links:
- link red_ball: geometry collision sphere radius=0.05; visual sphere radius=0.05
